Commit message: Codian URDF updates

File: urdf/codian.urdf (robot description, URDF)
Before this commit: robot codian, 15 links, 14 joints
Links:
- removed link con11_link
- removed link con22_link
- removed link con33_link
- added link A11, mass 0.00001; visual box size=0.01 0.01 0.01
- added link A12, mass 0.00001; visual box size=0.01 0.01 0.01
- added link A21, mass 0.00001; visual box size=0.01 0.01 0.01
- added link A22, mass 0.00001; visual box size=0.01 0.01 0.01
- added link A31, mass 0.00001; visual box size=0.01 0.01 0.01
- added link A32, mass 0.00001; visual box size=0.01 0.01 0.01
- link low_base: mass 0.00001 -> 0.001
Joints:
- removed joint con11
- removed joint con11_lleg_1
- removed joint con22
- removed joint con33
- added joint JA11: type revolute, parent low_base, child A11, origin xyz=0.052 -0.05 0 rpy=0 0 0, axis 1 0 0, limit lower=0 upper=0 effort=0 velocity=0
- added joint JA12: type revolute, parent low_base, child A12, origin xyz=-0.052 -0.05 0 rpy=0 0 0, axis 1 0 0, limit lower=0 upper=0 effort=0 velocity=0
- added joint JA21: type revolute, parent low_base, child A21, origin xyz=-0.01698 0.07059 0 rpy=0 0 4.1887902048, axis 1 0 0, limit lower=0 upper=0 effort=0 velocity=0
- added joint JA22: type revolute, parent low_base, child A22, origin xyz=-0.06962 -0.02059 0 rpy=0 0 4.1887902048, axis 1 0 0, limit lower=0 upper=0 effort=0 velocity=0
- added joint JA31: type revolute, parent low_base, child A31, origin xyz=0.06962 -0.02059 0 rpy=0 0 2.0943951024, axis 1 0 0, limit lower=0 upper=0 effort=0 velocity=0
- added joint JA32: type revolute, parent low_base, child A32, origin xyz=0.01698 0.07059 0 rpy=0 0 2.0943951024, axis 1 0 0, limit lower=0 upper=0 effort=0 velocity=0
- added joint base_spawn: type floating, parent base_link, child low_base, origin xyz=0 0 -0.710448 rpy=0 0 0
- joint con2_lleg_1: axis 1 1 1 -> -1 1 -1; mimic (none) -> joint=con_lleg_1; origin xyz=-0.052 -0.320 0 rpy=0 3.1415926536 0 -> xyz=-0.052 -0.320 0 rpy=2.555702653 0 3.141592654
- joint con2_lleg_2: axis 1 1 1 -> -1 1 -1; mimic (none) -> joint=con_lleg_2; origin xyz=-0.052 -0.320 0 rpy=0 3.1415926536 0 -> xyz=-0.052 -0.320 0 rpy=2.555702653 0 3.141592654
- joint con2_lleg_3: axis 1 1 1 -> -1 1 -1; mimic (none) -> joint=con_lleg_3; origin xyz=-0.052 -0.320 0 rpy=0 3.1415926536 0 -> xyz=-0.052 -0.320 0 rpy=2.555702653 0 3.141592654
- joint con_lleg_1: origin xyz=0.052 -0.320 0 rpy=0 0 0 -> xyz=0.052 -0.320 0 rpy=0.585890011 0 0
- joint con_lleg_2: origin xyz=0.052 -0.320 0 rpy=0 0 0 -> xyz=0.052 -0.320 0 rpy=0.585890011 0 0
- joint con_lleg_3: origin xyz=0.052 -0.320 0 rpy=0 0 0 -> xyz=0.052 -0.320 0 rpy=0.585890011 0 0
