Commit message: Code cleanup

File: urdf/delta_robot.urdf (robot description, URDF)
Before this commit: robot delta_robot, 19 links, 18 joints
Joints:
- joint base: origin xyz=0 0 1.359 rpy=0 0 0 -> xyz=0 0 1.5 rpy=0 0 0

Commit message: Updated files for codian robot (is now working)

File: urdf/delta_robot.urdf (robot description, URDF)
Before this commit: robot delta_robot, 19 links, 18 joints
Joints:
- joint con33_lleg_3: axis 0 1 0 -> 0 1zzz 0
