Commit message: Changed collision geomerty

File: urdf/conveyor.urdf (robot description, URDF)
Before this commit: robot simple_box, 1 links, 0 joints
Links:
- link my_box: geometry collision box size=10 10 0.1; visual mesh filename=/home/remco/catkin_ws/src/delta_robot_simulation/meshes/con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 scale=2 1 1
