Commit message: Smaller sphere, added maximum travel distance

File: urdf/object.urdf (robot description, URDF)
Before this commit: robot potato, 1 links, 0 joints
Links:
- link potato: geometry collision sphere radius=0.01; visual sphere radius=0.01

Commit message: Added rotation to objects

File: urdf/object.urdf (robot description, URDF)
Before this commit: robot potato, 1 links, 0 joints
Links:
- link potato: geometry collision box size=0.1 0.02 0.02; visual box size=0.1 0.02 0.02
